Commit message: Fix coverage navigation: update TF tree, center costmaps at (5,5), and add diff-drive plugin

File: src/moborobo_robot/description/robot_core.xacro (robot description, xacro)
@@ -113,6 +113,7 @@
     </collision>
     <inertial>
-      <mass value="0.5"/>
-      <inertia ixx="0.001266667" ixy="0" ixz="0" iyy="0.001266667" iyz="0" izz="0.0025"/>
+      <mass value="2"/>
+      <inertia ixx="0.005066668" ixy="0" ixz="0"
+             iyy="0.005066668" iyz="0" izz="0.01"/>
     </inertial>
   </link>
@@ -138,4 +139,28 @@
     </plugin>
   </gazebo>
+  <gazebo>
+    <plugin name="gazebo_ros_diff_drive" filename="libgazebo_ros_diff_drive.so">
+      <update_rate>50</update_rate>
+      <!-- Wheels -->
+      <left_joint>left_wheel_joint</left_joint>
+      <right_joint>right_wheel_joint</right_joint>
+      <!-- Kinematics -->
+      <wheel_separation>0.35</wheel_separation>   <!-- 2 × 0.175m from URDF -->
+      <wheel_diameter>0.2</wheel_diameter>         <!-- radius 0.1m × 2 -->
+      <!-- Limits -->
+      <max_wheel_torque>20</max_wheel_torque>
+      <max_wheel_acceleration>1.0</max_wheel_acceleration>
+      <!-- Topics -->
+      <command_topic>cmd_vel</command_topic>
+      <odometry_topic>odom</odometry_topic>
+      <odometry_frame>odom</odometry_frame>
+      <robot_base_frame>base_footprint</robot_base_frame>
+      <!-- TF -->
+      <publish_odom>true</publish_odom>
+      <publish_odom_tf>true</publish_odom_tf>      <!-- THIS publishes odom→base_footprint TF -->
+      <publish_wheel_tf>false</publish_wheel_tf>
+      <odometry_source>world</odometry_source>
+    </plugin>
+  </gazebo>
   <!-- Gazebo materials -->
   <gazebo reference="back_left_caster"><material>Gazebo/White</material></gazebo>
