Commit message: can now use zed camera to view point cloud, documentation later

File: src/moborobo_robot/description/camera.xacro (robot description, xacro)
@@ -1,4 +1,4 @@
 <?xml version="1.0"?>
-<robot xmlns:xacro="http://www.ros.org/wiki/xacro" >
+<robot xmlns:xacro="http://www.ros.org/wiki/xacro">
     <joint name="camera_joint" type="fixed">
         <parent link="base_link"/>
@@ -18,8 +18,9 @@
         <origin xyz="0 0 0" rpy="${-pi/2} 0 ${-pi/2}"/>
     </joint>
-    <link name="camera_link_optical"></link>
+    <link name="camera_link_optical"/>
+    <!-- UNCHANGED: RGB camera, keeps your existing /zed2/image_raw and /zed2/camera_info topics -->
     <gazebo reference="camera_link">
         <sensor name="camera" type="camera">
-            <pose> 0 0 0 0 0 0 </pose>
+            <pose>0 0 0 0 0 0</pose>
             <visualize>true</visualize>
             <update_rate>10</update_rate>
@@ -46,6 +47,42 @@
         </sensor>
     </gazebo>
+    <!-- CHANGED: Added a second Gazebo sensor for depth output -->
+    <gazebo reference="camera_link">
+        <!-- CHANGED: type is depth instead of normal RGB camera -->
+        <sensor name="depth_camera" type="depth">
+            <pose>0 0 0 0 0 0</pose>
+            <visualize>true</visualize>
+            <update_rate>10</update_rate>
+            <camera>
+                <horizontal_fov>1.089</horizontal_fov>
+                <!-- CHANGED: Depth images use float depth values, not RGB pixels -->
+                <image>
+                    <format>R_FLOAT32</format>
+                    <width>640</width>
+                    <height>480</height>
+                </image>
+                <clip>
+                    <near>0.05</near>
+                    <far>8.0</far>
+                </clip>
+            </camera>
+            <!-- CHANGED: Use libgazebo_ros_camera.so because your system does not have libgazebo_ros_depth_camera.so -->
+            <plugin name="depth_camera_controller" filename="libgazebo_ros_camera.so">
+                <ros>
+                    <!-- CHANGED: Namespace makes output topics start with /zed2/... -->
+                    <namespace>zed2</namespace>
+                    <!-- CHANGED: Depth image topic -->
+                    <remapping>~/image_raw:=depth/image_raw</remapping>
+                    <!-- CHANGED: Depth camera info topic -->
+                    <remapping>~/camera_info:=depth/camera_info</remapping>
+                </ros>
+                <!-- CHANGED: With namespace zed2 + camera_name depth, expected topics are /zed2/depth/image_raw and /zed2/depth/camera_info -->
+                <camera_name>depth</camera_name>
+                <frame_name>camera_link_optical</frame_name>
+            </plugin>
+        </sensor>
+    </gazebo>
     <gazebo reference="camera_link">
         <material>Gazebo/Black</material>
-      </gazebo>
+    </gazebo>
 </robot>
