Commit message: fix(simulation): update caster wheel physics, lock swivels, and shift gazebo arena

File: src/moborobo_robot/description/robot.urdf.xacro (robot description, xacro)
@@ -2,5 +2,4 @@
     <robot xmlns:xacro="http://www.ros.org/wiki/xacro"  name="moborobo_short">
         <xacro:include filename="robot_core.xacro" />
-        <xacro:include filename="controller.xacro" />
         <xacro:include filename="camera.xacro"/>
         <xacro:include filename="imu.xacro"/>

File: src/moborobo_robot/description/robot_core.xacro (robot description, xacro)
@@ -165,12 +165,36 @@
   <!-- Gazebo materials -->
   <gazebo reference="back_left_caster"><material>Gazebo/White</material></gazebo>
-  <gazebo reference="back_left_caster_wheel"><material>Gazebo/Black</material></gazebo>
+  <gazebo reference="back_left_caster_wheel">
+    <material>Gazebo/Black</material>
+    <mu1>0.0</mu1>
+    <mu2>0.0</mu2>
+  </gazebo>
   <gazebo reference="back_right_caster"><material>Gazebo/White</material></gazebo>
-  <gazebo reference="back_right_caster_wheel"><material>Gazebo/Black</material></gazebo>
+  <gazebo reference="back_right_caster_wheel">
+    <material>Gazebo/Black</material>
+    <mu1>0.0</mu1>
+    <mu2>0.0</mu2>
+  </gazebo>
   <gazebo reference="front_left_caster"><material>Gazebo/White</material></gazebo>
-  <gazebo reference="front_left_caster_wheel"><material>Gazebo/Black</material></gazebo>
+  <gazebo reference="front_left_caster_wheel">
+    <material>Gazebo/Black</material>
+    <mu1>0.0</mu1>
+    <mu2>0.0</mu2>
+  </gazebo>
   <gazebo reference="front_right_caster"><material>Gazebo/White</material></gazebo>
-  <gazebo reference="front_right_caster_wheel"><material>Gazebo/Black</material></gazebo>
-  <gazebo reference="left_wheel"><material>Gazebo/Black</material></gazebo>
-  <gazebo reference="right_wheel"><material>Gazebo/Black</material></gazebo>
+  <gazebo reference="front_right_caster_wheel">
+    <material>Gazebo/Black</material>
+    <mu1>0.0</mu1>
+    <mu2>0.0</mu2>
+  </gazebo>
+  <gazebo reference="left_wheel">
+    <material>Gazebo/Black</material>
+    <mu1>1.0</mu1>
+    <mu2>1.0</mu2>
+  </gazebo>
+  <gazebo reference="right_wheel">
+    <material>Gazebo/Black</material>
+    <mu1>1.0</mu1>
+    <mu2>1.0</mu2>
+  </gazebo>
 </robot>
