Commit message: fix: fixed the lidar obstructing the camera. added oak d pro to the sim

File: src/moborobo_robot/description/lidar.xacro (robot description, xacro)
@@ -5,5 +5,5 @@
         <parent link="base_link"/>
         <child link="lidar"/>
-        <origin xyz="0.2 0 0.6" rpy="0 0 0"/>
+        <origin xyz="0.05 0 0.6" rpy="0 0 0"/>
     </joint>
     <link name="lidar">

File: src/moborobo_robot/description/robot.urdf.xacro (robot description, xacro)
@@ -3,7 +3,9 @@
         <xacro:include filename="robot_core.xacro" />
         <xacro:include filename="controller.xacro" />
-        <xacro:include filename="camera.xacro"/>
-        <xacro:include filename="imu.xacro"/>
-        <xacro:include filename="lidar.xacro"/>
+        <xacro:include filename="oak_d_pro.xacro"/>
+        <!-- commenting this out because it's not needed for now, oak camera supplies all -->
+        <!-- <xacro:include filename="camera.xacro"/> -->
+        <!-- <xacro:include filename="imu.xacro"/> -->
+        <!-- <xacro:include filename="lidar.xacro"/> -->
         <!-- <xacro:include filename="gps.xacro"/> -->
     </robot>
